File: oscillator_prototype.kicad_pcb (KiCad board)
At the start: 2 copper layers, 90 x 104 mm, 94 parts, among them J1 shark fin, J10 Conn_01x06_Male, J11 Conn_01x06_Female, J12 Conn_01x06_Male, J13 Conn_01x06_Female, J14 Conn_01x06_Male, J3 1v/oct, J4 Triangle, J6 Sync, J7 Eurorack power, J8 Linear FM, J9 Conn_01x06_Female, Q1 MMBT3904, Q2 MMBT3906, Q3 BC857BS, Q4 MMBT3904, Q5 MMBT3904, SW1 Sync Mode, U1 LT1013-SOIC, U10 LM4040AIM3-5, U11 LM4040AIM3-5, U2 TL074, U3 LM13700, U4 LM311, U5 LM4040AIM3-2.5, U6 DG418, U7 LM311, U8 LM4040AIM3-2.5, U9 LM4040AIM3-2.5

Commit message: Add all missing component values to schematic
Parts:
- C3: value C_Small -> 1n
- R11, R17, R19, R24: value R_Small_US -> 18k
- R18: value R_Small_US -> 24k
- R20: value R_Small_US -> 240k
- R28, R32: value R_Small_US -> 3k3
- R29: value R_Small_US -> 2M2
- R3: value ??k -> 47k
- R30: value R_Small_US -> 270R
- R31: value R_Small_US -> 820k
- R4: value Xk yyy ppm -> 2k +3300ppm/C
- R6: value ??k -> 750k
- R8: value R_Small_US -> 390R
- RV3: value R_POT_TRIM_US -> 100R
- RV6: value R_POT_TRIM_US -> 100k
