File: oscillator_prototype.sch (KiCad schematic (older format))
At the start: 99 parts, among them J1 shark fin, J2 Exp FM, J3 1v/oct, J4 Triangle, J5 Pulse, J6 Sync, J7 Eurorack power, J8 Linear FM, J9 PWM, Q1 MMBT3904, Q2 MMBT3906, Q3 BC857BS, Q4 MMBT3904, Q5 MMBT3904, SW1 Sync Mode, SW2 Audio/LFO, U1 LT1013, U2 TL074, U3 LM13700, U4 LM311, U5 LM311, U6 DG418, U7 LM311, U8 TL072

Commit message: Switch to SMT resistors/caps/diodes (mostly)
Parts:
- C1: footprint Capacitor_THT:C_Disc_D5.0mm_W2.5mm_P5.00mm -> Capacitor_SMD:C_0603_1608Metric_Pad1.08x0.95mm_HandSolder
- C10, C11, C12, C13, C14, C15, C16, C17, C19, C20, C21, C22, C23, C24, C25, C26, C3, C4, C5, C7, C8: footprint Capacitor_THT:C_Disc_D5.0mm_W2.5mm_P5.00mm -> Capacitor_SMD:C_0805_2012Metric_Pad1.18x1.45mm_HandSolder
- D1, D2, D3: footprint Diode_THT:D_DO-35_SOD27_P7.62mm_Horizontal -> Diode_SMD:D_0805_2012Metric_Pad1.15x1.40mm_HandSolder
- R1, R10, R11, R12, R13, R14, R15, R16, R17, R18, R19, R2, R20, R21, R22, R23, R24, R25, R26, R27, R28, R29, R3, R30, R31, R32, R33, R34, R5, R6, R7, R8, R9: footprint Resistor_THT:R_Axial_DIN0204_L3.6mm_D1.6mm_P5.08mm_Horizontal -> Resistor_SMD:R_0805_2012Metric_Pad1.20x1.40mm_HandSolder
- R4: footprint Resistor_THT:R_Axial_DIN0207_L6.3mm_D2.5mm_P7.62mm_Horizontal -> Resistor_THT:R_Axial_DIN0204_L3.6mm_D1.6mm_P5.08mm_Horizontal

Commit message: Complete layout
Parts:
- removed C16, C17, C25, C26, C7, C8: 100n, Capacitor_SMD:C_0805_2012Metric_Pad1.18x1.45mm_HandSolder, symbol Device:C_Small
- removed J2: Exp FM, kicad_libraries:Jack_3.5mm_QingPu_WQP-PJ398SM_Vertical_CircularHoles-translated, symbol Synth:AudioJack1_SwitchT
- removed J5: Pulse, kicad_libraries:Jack_3.5mm_QingPu_WQP-PJ398SM_Vertical_CircularHoles-translated, symbol Synth:AudioJack1_SwitchT
- removed J9: PWM, kicad_libraries:Jack_3.5mm_QingPu_WQP-PJ398SM_Vertical_CircularHoles-translated, symbol Synth:AudioJack1_SwitchT
- removed R34: 100k, Resistor_SMD:R_0805_2012Metric_Pad1.20x1.40mm_HandSolder, symbol Device:R_Small_US
- removed RV4, RV9: 100k, kicad_libraries:Potentiometer_Alpha_RD901F-40-00D_Single_Vertical-translated, symbol Device:R_POT_US
- removed RV8: B100k, kicad_libraries:Potentiometer_Alpha_RD901F-40-00D_Single_Vertical-translated, symbol Device:R_POT_US
- removed SW2: Audio/LFO, ljwall-kicad-footprints:Dailywell_sub-mini_toggle_DPDT, symbol Switch:SW_Push_DPDT
- removed U1: LT1013, Package_SO:SOIC-8_3.9x4.9mm_P1.27mm, symbol Amplifier_operational_extended:LT1013
- removed U5: LM311, Package_SO:SOIC-8_3.9x4.9mm_P1.27mm, symbol Comparator:LM311
- removed U8: TL072, Package_SO:SOIC-8_3.9x4.9mm_P1.27mm, symbol Amplifier_Operational:TL072
- added D6, D7, D8, D9: 1N4148, Diode_SMD:D_0805_2012Metric_Pad1.15x1.40mm_HandSolder, symbol Device:D_Small
- added J10, J12, J14: Conn_01x06_Male, Connector_PinHeader_2.54mm:PinHeader_1x06_P2.54mm_Vertical, symbol Connector:Conn_01x06_Male
- added J11, J13, J9: Conn_01x06_Female, Connector_PinHeader_2.54mm:PinHeader_1x06_P2.54mm_Vertical, symbol Connector:Conn_01x06_Female
- added RV4: 2k, Potentiometer_THT:Potentiometer_Bourns_3266X_Horizontal, symbol Device:R_POT_TRIM_US
- added TP1: vref, TestPoint:TestPoint_Pad_D2.0mm, symbol Connector:TestPoint
- added U1, U5: LT1013-SOIC, Package_SO:SOIC-8_3.9x4.9mm_P1.27mm, symbol ljw-kicad-symbols:LT1013-SOIC
- added U8: LM336Z-5.0, Package_TO_SOT_THT:TO-92_Inline, symbol Reference_Voltage:LM385Z-ADJ
- C1: value C_Small -> 1n; footprint Capacitor_SMD:C_0603_1608Metric_Pad1.08x0.95mm_HandSolder -> Capacitor_SMD:C_0805_2012Metric_Pad1.18x1.45mm_HandSolder
- C5: value 10n -> 100n
- C6: value 470n (polyester) -> 100n; footprint Capacitor_THT:C_Rect_L7.2mm_W3.5mm_P5.00mm_FKS2_FKP2_MKS2_MKP2 -> Capacitor_SMD:C_0805_2012Metric_Pad1.18x1.45mm_HandSolder
- J7: footprint Connector_IDC:IDC-Header_2x05_P2.54mm_Vertical -> Connector_IDC:IDC-Header_2x05_P2.54mm_Horizontal
- R10, R14: value R_Small_US -> 100k
- R17: value 20k -> 120k
- R19: value 1k -> 3k6
- R24: value 1k -> 10k
- R28: value 1k -> 4k7
- R3: value R_Small_US -> 68k
- R32: value 100k -> 10k
- R33: value 100k -> 4k7
- R6: value R_Small_US -> 680k
- RV1, RV2: value 100k -> 50k
Connections:
- net +12V: now also C5.1, C6.1, R19.1, U1.6 (v+), U5.6 (v+); no longer C15.1, U3.10, U3.7, U3.8, U3.9
- net +5V: now also J10.3 (Pin_3), J10.4 (Pin_4), U5.7, U5.8 (-); no longer R17.2, RV1.3, RV2.3
- net -12V: now also C15.2, U1.2 (v-), U5.2 (v-)
- net -5V: now also R17.2, R24.2, RV5.3, U5.5; no longer RV1.1, RV5.1
- net GND: now also C15.1, C5.2, C6.2, U2.12 (+), U2.5 (+), D8.1 (K), J10.5 (Pin_5), J10.6 (Pin_6), J12.3 (Pin_3), J12.5 (Pin_5), J12.6 (Pin_6), J14.5 (Pin_5), J14.6 (Pin_6), U1.1 (+), U1.3 (+), U5.3 (+), U8.3 (A); no longer C15.2, J1.S, J3.S, J3.TN, J4.S, J6.S, J6.TN, J8.S, J8.TN, RV2.1, RV7.1, U2.3 (+)
- net TC_a: now also R30.1, U2.13 (-), U3.5; no longer U3.12, U6.1
- net TC_b: now also U2.14, U2.3 (+), U6.1; no longer C6.2, R28.1, R30.1, U2.12 (+)
- net at C3.1, D1.1 (K), D3.2 (A)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: now also U1.5
- net at C3.2, Q3.3 (C2), R20.1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: now also U1.4 (-)
- net at C1.2, R14.1, R29.2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: now also R17.1, U1.8 (-); no longer R10.1
- net at C1.1, R4.1, RV3.1: now also U1.7
- net at U3.16: now also Q2.3 (C); no longer Q3.6 (C1)
- net at U3.1: now also Q3.6 (C1); no longer Q2.3 (C)
- net at R1.2, R2.1, U2.9 (-): now also U3.12; no longer U3.5
- net at R20.2, RV5.2: now also RV5.1; no longer RV5.3
- net at R28.2: now also RV4.3
- net switch_a_f: now reaches SW1.2 (B)
- net switch_a_f: now also J9.1 (Pin_1); no longer U7.1 (GND)
- net at U2.6 (-), U2.7: no longer R19.1
- net at R19.2: now also R32.1, D6.2 (A), TP1.1, U5.1 (+), U8.2 (K)
- net at R10.2: now also RV2.3
- net v_per_oct_f: now reaches J3.T
- net v_per_oct_f: now also J13.3 (Pin_3); no longer R14.2
- net switch_b_m: now reaches R23.1, U6.6
- net switch_b_m: now also J12.4 (Pin_4); no longer SW1.1 (A)
- net coarse_f: now reaches RV1.2
- net coarse_f: now also J13.2 (Pin_2); no longer R3.2
- net fine_f: now reaches RV2.2
- net fine_f: now also J13.1 (Pin_1); no longer R6.2
- net at U2.1: now also R16.1, U2.2 (-); no longer R32.1
- net saw_f: now reaches J1.T
- net saw_f: now also J11.1 (Pin_1); no longer R5.2
- net tri_f: now reaches J4.T
- net tri_f: now also J11.2 (Pin_2); no longer R16.2
- net lin_fm_f: now reaches RV7.2
- net lin_fm_f: now also J13.4 (Pin_4); no longer R31.2
- net at R33.2: now also D9.2 (A)
- removed net SC_a: C4.2, C5.2, J6.T, R24.1
- net SC_b: no longer names the net of C4.1, D2.1 (K), Q4.1 (B), R25.1
- new net: U3.10, U3.9
- new net: U3.7, U3.8
- new net: D8.2 (A), D9.1 (K)
- new net: R33.1, RV4.1
- new net: RV4.2, U8.1 (FB)
- new net: D7.1 (K), R28.1
- new net: D6.1 (K), D7.2 (A)
- new net: R24.1, R32.2, U5.4 (-)
- new net 5V_f: J9.3 (Pin_3), J9.4 (Pin_4), R10.1, RV1.3
- new net GND_f: J1.S, J11.3 (Pin_3), J11.5 (Pin_5), J11.6 (Pin_6), J13.5 (Pin_5), J13.6 (Pin_6), J3.S, J3.TN, J4.S, J6.S, J6.TN, J8.S, J8.TN, J9.5 (Pin_5), J9.6 (Pin_6), RV1.1, RV2.1, RV7.1
- new net coarse_m: J14.2 (Pin_2), R3.2
- new net fine_m: J14.1 (Pin_1), R6.2
- new net lin_fm_m: J14.4 (Pin_4), R31.2
- new net saw_m: J12.1 (Pin_1), R5.2
- new net switch_a_m: J10.1 (Pin_1), U7.1 (GND)
- new net switch_b_f: J11.4 (Pin_4), SW1.1 (A)
- new net sync_f: J6.T, J9.2 (Pin_2)
- new net sync_m: C4.2, J10.2 (Pin_2)
- new net tri_m: J12.2 (Pin_2), R16.2
- new net v_per_oct_m: J14.3 (Pin_3), R14.2
- no-connect marks 12 -> 9
Other:
- moved on the sheet: C10, C11, C12, C13, C14, C18, C19, C20, C21, C22, C23, C4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

Commit message: Refactor layout and simplify circuit
Parts:
- removed C24: 100n, Capacitor_SMD:C_0805_2012Metric_Pad1.18x1.45mm_HandSolder, symbol Device:C_Small
- removed D6, D7, D8, D9: 1N4148, Diode_SMD:D_0805_2012Metric_Pad1.15x1.40mm_HandSolder, symbol Device:D_Small
- removed JP1: Jumper_NC_Dual, Connector_PinHeader_2.54mm:PinHeader_1x03_P2.54mm_Vertical, symbol Device:Jumper_NC_Dual
- removed R10: 100k, Resistor_SMD:R_0805_2012Metric_Pad1.20x1.40mm_HandSolder, symbol Device:R_Small_US
- removed R33: 4k7, Resistor_SMD:R_0805_2012Metric_Pad1.20x1.40mm_HandSolder, symbol Device:R_Small_US
- removed RV4: 2k, Potentiometer_THT:Potentiometer_Bourns_3266X_Horizontal, symbol Device:R_POT_TRIM_US
- removed RV5: R_POT_TRIM_US, Potentiometer_THT:Potentiometer_Bourns_3266X_Horizontal, symbol Device:R_POT_TRIM_US
- removed U5: LT1013-SOIC, Package_SO:SOIC-8_3.9x4.9mm_P1.27mm, symbol ljw-kicad-symbols:LT1013-SOIC
- removed U8: LM336Z-5.0, Package_TO_SOT_THT:TO-92_Inline, symbol Reference_Voltage:LM385Z-ADJ
- added C16, C17, C7, C8: 100n, Capacitor_SMD:C_0805_2012Metric_Pad1.18x1.45mm_HandSolder, symbol Device:C_Small
- added U10, U11: LM4040AIM3-5, Package_TO_SOT_SMD:SOT-23, symbol Reference_Voltage:LM4040DBZ-2.5
- added U5, U8, U9: LM4040AIM3-2.5, Package_TO_SOT_SMD:SOT-23, symbol Reference_Voltage:LM4040DBZ-2.5
- C2: value 1n Mica -> 1n C0G; footprint ljwall-kicad-footprints:Cornell-Dubilier_CD15_Mica_Capacitor_L16.5mm_T5.6mm_P8.7mm -> Capacitor_SMD:C_0805_2012Metric_Pad1.18x1.45mm_HandSolder
- R17: value 120k -> R_Small_US
- R19: value 3k6 -> R_Small_US
- R24, R32: value 10k -> R_Small_US
- R28: value 4k7 -> R_Small_US
- R3: value 68k -> ??k
- R6: value 680k -> ??k
- TP1: value vref -> TestPoint; footprint TestPoint:TestPoint_Pad_D2.0mm -> TestPoint:TestPoint_Pad_2.5x2.5mm
Connections:
- net +12V: now also J10.6 (Pin_6), R28.1, C16.1; no longer C11.1, R19.1
- net +5V: now also R28.2, U10.1 (K); no longer J10.3 (Pin_3), J10.4 (Pin_4)
- net -12V: now also J12.1 (Pin_1), R17.2, R32.2, C17.2, C7.2
- net -5V: now also R32.1, U11.2 (A); no longer R17.2, R24.2
- net GND: now also J10.3 (Pin_3), J10.4 (Pin_4), J12.4 (Pin_4), C16.2, C17.1, C7.1, U10.2 (A), U11.1 (K), U5.1 (K); no longer C11.2, J10.6 (Pin_6), J12.3 (Pin_3), J12.6 (Pin_6)
- net GND_f: now also C11.2, J11.4 (Pin_4), J9.3 (Pin_3), J9.4 (Pin_4), C8.1, U8.1 (K), U9.2 (A); no longer J11.3 (Pin_3), J11.6 (Pin_6), J9.6 (Pin_6), RV1.1
- net saw_f: now also J11.6 (Pin_6); no longer J11.1 (Pin_1)
- net saw_m: now also J12.6 (Pin_6); no longer J12.1 (Pin_1)
- net switch_a_f: now also J9.2 (Pin_2); no longer J9.1 (Pin_1)
- net switch_a_m: now also J10.2 (Pin_2); no longer J10.1 (Pin_1)
- net switch_b_f: now also J11.3 (Pin_3); no longer J11.4 (Pin_4)
- net switch_b_m: now also J12.3 (Pin_3); no longer J12.4 (Pin_4)
- net sync_f: now also J9.1 (Pin_1); no longer J9.2 (Pin_2)
- net sync_m: now also J10.1 (Pin_1); no longer J10.2 (Pin_2)
- net at R20.2: now also R17.1, U5.2 (A)
- net at C1.1, R4.1, RV3.1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: now also TP1.1
- net at RV3.2: now also Q3.2 (B1)
- net at C1.2, R14.1, R29.2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: no longer R17.1
- net 2.5V_f: now reaches RV2.3
- net 2.5V_f: now also R19.2, RV1.3, U9.1 (K)
- net -2.5V_f: now reaches R24.1
- net -2.5V_f: now also RV1.1, U8.2 (A); no longer R32.2
- removed net 5V_f: J9.3 (Pin_3), J9.4 (Pin_4), RV1.3
- new net -12V_f: C8.2, J11.1 (Pin_1), R24.2
- new net 12V_f: C11.1, J9.6 (Pin_6), R19.1
Other:
- moved on the sheet: C4, D2, J10, J11, J12, J13, J14, J6, J9, Q4, Q5, R20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
